File: Replica_Reles.sch (KiCad schematic (older format))
At the start: 66 parts, among them J1 Tira de Pines Macho, J2 Bornera, J3 Bornera, J4 Bornera, J5 Bornera, J6 Bornera, J7 Bornera, J8 Bornera, J9 Bornera, K1 SONGLE_SRD_Form_C, K2 SONGLE_SRD_Form_C, K3 SONGLE_SRD_Form_C, K4 SONGLE_SRD_Form_C, K5 SONGLE_SRD_Form_C, K6 SONGLE_SRD_Form_C, K7 SONGLE_SRD_Form_C, K8 SONGLE_SRD_Form_C, Q1 S8050, Q2 S8050, Q3 S8050, Q4 S8050, Q5 S8050, Q6 S8050, Q7 S8050, Q8 S8050, U1 PC817, U2 PC817, U3 PC817, U4 PC817, U5 PC817, U6 PC817, U7 PC817, U8 PC817

Commit message: Inicio PCB: Posicionamiento de Componentes
Parts:
- added MH1, MH2, MH3, MH4: MountingHole, MountingHole:MountingHole_3.2mm_M3_ISO14580, symbol Mechanical:MountingHole
- J1: renamed from J4; footprint TerminalBlock:TerminalBlock_Altech_AK300-3_P5.00mm -> TerminalBlock:TerminalBlock_bornier-3_P5.08mm
- J2: renamed from J7; footprint TerminalBlock:TerminalBlock_Altech_AK300-3_P5.00mm -> TerminalBlock:TerminalBlock_bornier-3_P5.08mm
- J3: renamed from J1; footprint Connector_PinSocket_2.54mm:PinSocket_1x10_P2.54mm_Vertical -> Connector_PinHeader_2.54mm:PinHeader_1x10_P2.54mm_Vertical
- J4: renamed from J2; footprint TerminalBlock:TerminalBlock_Altech_AK300-3_P5.00mm -> TerminalBlock:TerminalBlock_bornier-3_P5.08mm
- J5, J9: footprint TerminalBlock:TerminalBlock_Altech_AK300-3_P5.00mm -> TerminalBlock:TerminalBlock_bornier-3_P5.08mm
- J6: renamed from J8; footprint TerminalBlock:TerminalBlock_Altech_AK300-3_P5.00mm -> TerminalBlock:TerminalBlock_bornier-3_P5.08mm
- J7: renamed from J3; footprint TerminalBlock:TerminalBlock_Altech_AK300-3_P5.00mm -> TerminalBlock:TerminalBlock_bornier-3_P5.08mm
- J8: renamed from J6; footprint TerminalBlock:TerminalBlock_Altech_AK300-3_P5.00mm -> TerminalBlock:TerminalBlock_bornier-3_P5.08mm
- renumbered D6 to D1, D14 to D2, D4 to D3, D9 to D4, D15 to D5, D5 to D6, D10 to D7, D16 to D8, D3 to IN1, D11 to IN2, D1 to IN3, D7 to IN4, D12 to IN5, D2 to IN6, D8 to IN7, D13 to IN8, K3 to K1, K6 to K2, K1 to K3, K7 to K5, K2 to K6, K5 to K7, Q3 to Q1, Q6 to Q2, Q1 to Q3, Q7 to Q5, Q2 to Q6, Q5 to Q7, R5 to R1, R15 to R10, R2 to R11, R4 to R12, R8 to R13, R10 to R14, R13 to R15, R6 to R2, R11 to R3, R14 to R4, R1 to R5, R3 to R6, R9 to R8, R12 to R9, U3 to U1, U6 to U2, U1 to U3, U7 to U5, U2 to U6, U5 to U7
Connections:
- wire segments 287 -> 291
Other:
- note added: "AGUJEROS DE SUJECION DE LA PLACA\n"
- note added: "Rele n°1\n\n"
- note added: "Rele n°5\n"
- note added: "Rele n°6\n"
- note added: "Rele n°7\n"
- note added: "Rele n°8\n\n"
- note removed: "Rele n°1\n"
- note removed: "Rele n°5"
- note removed: "Rele n°6"
- note removed: "Rele n°7"
- note removed: "Rele n°8\n"

Commit message: Cambios en posicionamiento, ruteo y mas documentacion
Parts:
- removed JP1: VCC JD-VCC, Connector_PinHeader_2.54mm:PinHeader_1x02_P2.54mm_Vertical, symbol Device:Jumper
- added J10: Conn_01x03, Connector_PinHeader_2.54mm:PinHeader_1x03_P2.54mm_Vertical, symbol Connector_Generic:Conn_01x03
- K1, K2, K3, K4, K5, K6, K7, K8: footprint Relay_THT:Relay_SPDT_SANYOU_SRD_Series_Form_C -> Relay_THT:Relay_SPDT_SONGLE_SRD_Series_Form_C
- Q1, Q2, Q3, Q4, Q5, Q6, Q7, Q8: symbol Transistor_BJT:S8050 -> Device:Q_NPN_BEC
Connections:
- wire segments 291 -> 293
Changed lines of the file:
@@
 $EndComp
 $Comp
-L Transistor_BJT:S8050 Q1
+L Device:Q_NPN_BEC Q1
 U 1 1 5BA4F7BD
 P 3950 1950
@@
 	1    800  1400
 	-1   0    0    -1
-$EndComp
-$Comp
-L Device:Jumper JP1
-U 1 1 5BA50437
-P 1200 7050
-F 0 "JP1" H 1200 7314 50  0000 C CNN
-F 1 "VCC      JD-VCC" H 1250 7200 50  0000 C CNN
-F 2 "Connector_PinHeader_2.54mm:PinHeader_1x02_P2.54mm_Vertical" H 1200 7050 50  0001 C CNN
-F 3 "~" H 1200 7050 50  0001 C CNN
-	1    1200 7050
-	1    0    0    -1
 $EndComp
 $Comp
@@
 F 0 "K1" H 4250 1800 50  0000 L CNN
 F 1 "SONGLE_SRD_Form_C" H 3950 1700 50  0000 L CNN
-F 2 "Relay_THT:Relay_SPDT_SANYOU_SRD_Series_Form_C" H 4700 1250 50  0001 L CNN
+F 2 "Relay_THT:Relay_SPDT_SONGLE_SRD_Series_Form_C" H 4700 1250 50  0001 L CNN
 F 3 "http://www.sanyourelay.ca/public/products/pdf/SRD.pdf" H 4250 1300 50  0001 C CNN
 	1    4250 1300
@@
 $EndComp
 $Comp
-L Transistor_BJT:S8050 Q2
+L Device:Q_NPN_BEC Q2
 U 1 1 5BC08FFC
 P 8700 1950
@@
 F 0 "K2" H 9000 1800 50  0000 L CNN
 F 1 "SONGLE_SRD_Form_C" H 8700 1700 50  0000 L CNN
-F 2 "Relay_THT:Relay_SPDT_SANYOU_SRD_Series_Form_C" H 9450 1250 50  0001 L CNN
+F 2 "Relay_THT:Relay_SPDT_SONGLE_SRD_Series_Form_C" H 9450 1250 50  0001 L CNN
 F 3 "http://www.sanyourelay.ca/public/products/pdf/SRD.pdf" H 9000 1300 50  0001 C CNN
 	1    9000 1300
@@
 $EndComp
 $Comp
-L Transistor_BJT:S8050 Q3
+L Device:Q_NPN_BEC Q3
 U 1 1 5BC0CC95
 P 2650 4050
@@
 F 0 "K3" H 2950 3900 50  0000 L CNN
 F 1 "SONGLE_SRD_Form_C" H 2650 3800 50  0000 L CNN
-F 2 "Relay_THT:Relay_SPDT_SANYOU_SRD_Series_Form_C" H 3400 3350 50  0001 L CNN
+F 2 "Relay_THT:Relay_SPDT_SONGLE_SRD_Series_Form_C" H 3400 3350 50  0001 L CNN
 F 3 "http://www.sanyourelay.ca/public/products/pdf/SRD.pdf" H 2950 3400 50  0001 C CNN
 	1    2950 3400
@@
 $EndComp
 $Comp
-L Transistor_BJT:S8050 Q4
+L Device:Q_NPN_BEC Q4
 U 1 1 5BC1910B
 P 6050 4050
@@
 F 0 "K4" H 6350 3900 50  0000 L CNN
 F 1 "SONGLE_SRD_Form_C" H 6050 3800 50  0000 L CNN
-F 2 "Relay_THT:Relay_SPDT_SANYOU_SRD_Series_Form_C" H 6800 3350 50  0001 L CNN
+F 2 "Relay_THT:Relay_SPDT_SONGLE_SRD_Series_Form_C" H 6800 3350 50  0001 L CNN
 F 3 "http://www.sanyourelay.ca/public/products/pdf/SRD.pdf" H 6350 3400 50  0001 C CNN
 	1    6350 3400
@@
 $EndComp
 $Comp
-L Transistor_BJT:S8050 Q5
+L Device:Q_NPN_BEC Q5
 U 1 1 5BC1FA57
 P 9500 4050
@@
 F 0 "K5" H 9800 3900 50  0000 L CNN
 F 1 "SONGLE_SRD_Form_C" H 9500 3800 50  0000 L CNN
-F 2 "Relay_THT:Relay_SPDT_SANYOU_SRD_Series_Form_C" H 10250 3350 50  0001 L CNN
+F 2 "Relay_THT:Relay_SPDT_SONGLE_SRD_Series_Form_C" H 10250 3350 50  0001 L CNN
 F 3 "http://www.sanyourelay.ca/public/products/pdf/SRD.pdf" H 9800 3400 50  0001 C CNN
 	1    9800 3400
@@
 $EndComp
 $Comp
-L Transistor_BJT:S8050 Q6
+L Device:Q_NPN_BEC Q6
 U 1 1 5BC7F002
 P 2650 5850
@@
 F 0 "K6" H 2950 5700 50  0000 L CNN
 F 1 "SONGLE_SRD_Form_C" H 2650 5600 50  0000 L CNN
-F 2 "Relay_THT:Relay_SPDT_SANYOU_SRD_Series_Form_C" H 3400 5150 50  0001 L CNN
+F 2 "Relay_THT:Relay_SPDT_SONGLE_SRD_Series_Form_C" H 3400 5150 50  0001 L CNN
 F 3 "http://www.sanyourelay.ca/public/products/pdf/SRD.pdf" H 2950 5200 50  0001 C CNN
 	1    2950 5200
@@
 $EndComp
 $Comp
-L Transistor_BJT:S8050 Q7
+L Device:Q_NPN_BEC Q7
 U 1 1 5BC7F076
 P 6050 5850
@@
 F 0 "K7" H 6350 5700 50  0000 L CNN
 F 1 "SONGLE_SRD_Form_C" H 6050 5600 50  0000 L CNN
-F 2 "Relay_THT:Relay_SPDT_SANYOU_SRD_Series_Form_C" H 6800 5150 50  0001 L CNN
+F 2 "Relay_THT:Relay_SPDT_SONGLE_SRD_Series_Form_C" H 6800 5150 50  0001 L CNN
 F 3 "http://www.sanyourelay.ca/public/products/pdf/SRD.pdf" H 6350 5200 50  0001 C CNN
 	1    6350 5200
@@
 $EndComp
 $Comp
-L Transistor_BJT:S8050 Q8
+L Device:Q_NPN_BEC Q8
 U 1 1 5BC7F0EA
 P 9500 5850
@@
 F 0 "K8" H 9800 5700 50  0000 L CNN
 F 1 "SONGLE_SRD_Form_C" H 9500 5600 50  0000 L CNN
-F 2 "Relay_THT:Relay_SPDT_SANYOU_SRD_Series_Form_C" H 10250 5150 50  0001 L CNN
+F 2 "Relay_THT:Relay_SPDT_SONGLE_SRD_Series_Form_C" H 10250 5150 50  0001 L CNN
 F 3 "http://www.sanyourelay.ca/public/products/pdf/SRD.pdf" H 9800 5200 50  0001 C CNN
 	1    9800 5200
@@
 Wire Notes Line
 	1900 6500 550  6500
-Wire Wire Line
-	900  7050 700  7050
-Wire Wire Line
-	700  7050 700  6850
-$Comp
-L power:+5V #PWR019
-U 1 1 5BD1FFBA
-P 700 6850
-F 0 "#PWR019" H 700 6700 50  0001 C CNN
-F 1 "+5V" H 715 7023 50  0000 C CNN
-F 2 "" H 700 6850 50  0001 C CNN
-F 3 "" H 700 6850 50  0001 C CNN
-	1    700  6850
-	1    0    0    -1
-$EndComp
-Text Label 1800 7050 2    50   ~ 0
+Text Label 1250 6850 2    50   ~ 0
 JD-VCC
-Wire Wire Line
-	1500 7050 1800 7050
 Wire Wire Line
 	1900 4750 2100 4750
@@
 Text Label 5300 2950 0    50   ~ 0
 JD-VCC
-Text Notes 850  7400 0    50   ~ 10
-JUMPER \nALIMENTACION RELES \nA VCC\n
 Wire Notes Line
 	6200 500  6200 2450
@@
 Text Notes 3300 7600 0    50   ~ 10
 AGUJEROS DE SUJECION DE LA PLACA\n
+Text Notes 1100 7550 0    50   ~ 10
+JUMPER \nALIMENTACION RELES \nA VCC\n
+$Comp
+L Connector_Generic:Conn_01x03 J10
+U 1 1 5BB7A675
+P 750 6950
+F 0 "J10" H 670 7267 50  0000 C CNN
+F 1 "Conn_01x03" H 670 7176 50  0000 C CNN
+F 2 "Connector_PinHeader_2.54mm:PinHeader_1x03_P2.54mm_Vertical" H 750 6950 50  0001 C CNN
+F 3 "~" H 750 6950 50  0001 C CNN
+	1    750  6950
+	-1   0    0    -1
+$EndComp
+Wire Wire Line
+	950  6950 1650 6950
+Wire Wire Line
+	1650 6950 1650 6850
+$Comp
+L power:+5V #PWR0101
+U 1 1 5BBFDDD1
+P 1650 6850
+F 0 "#PWR0101" H 1650 6700 50  0001 C CNN
+F 1 "+5V" H 1665 7023 50  0000 C CNN
+F 2 "" H 1650 6850 50  0001 C CNN
+F 3 "" H 1650 6850 50  0001 C CNN
+	1    1650 6850
+	1    0    0    -1
+$EndComp
+Wire Wire Line
+	950  6850 1250 6850
+Wire Wire Line
+	950  7050 1650 7050
+Wire Wire Line
+	1650 7050 1650 7150
+$Comp
+L power:GND #PWR0102
+U 1 1 5BC5719E
+P 1650 7150
+F 0 "#PWR0102" H 1650 6900 50  0001 C CNN
+F 1 "GND" H 1655 6977 50  0000 C CNN
+F 2 "" H 1650 7150 50  0001 C CNN
+F 3 "" H 1650 7150 50  0001 C CNN
+	1    1650 7150
+	1    0    0    -1
+$EndComp
 $EndSCHEMATC

Commit message: Arreglos menores y agregado de documentacion
Changed lines of the file:
@@
 L Mechanical:MountingHole MH1
 U 1 1 5BAA4418
-P 3250 6850
-F 0 "MH1" H 3350 6896 50  0000 L CNN
-F 1 "MountingHole" H 3350 6805 50  0000 L CNN
-F 2 "MountingHole:MountingHole_3.2mm_M3_ISO14580" H 3250 6850 50  0001 C CNN
-F 3 "~" H 3250 6850 50  0001 C CNN
-	1    3250 6850
+P 2450 6750
+F 0 "MH1" H 2550 6796 50  0000 L CNN
+F 1 "MountingHole" H 2550 6705 50  0000 L CNN
+F 2 "MountingHole:MountingHole_3.2mm_M3_ISO14580" H 2450 6750 50  0001 C CNN
+F 3 "~" H 2450 6750 50  0001 C CNN
+	1    2450 6750
 	1    0    0    -1
 $EndComp
@@
 L Mechanical:MountingHole MH2
 U 1 1 5BAA49A8
-P 4200 6850
-F 0 "MH2" H 4300 6896 50  0000 L CNN
-F 1 "MountingHole" H 4300 6805 50  0000 L CNN
-F 2 "MountingHole:MountingHole_3.2mm_M3_ISO14580" H 4200 6850 50  0001 C CNN
-F 3 "~" H 4200 6850 50  0001 C CNN
-	1    4200 6850
+P 3400 6750
+F 0 "MH2" H 3500 6796 50  0000 L CNN
+F 1 "MountingHole" H 3500 6705 50  0000 L CNN
+F 2 "MountingHole:MountingHole_3.2mm_M3_ISO14580" H 3400 6750 50  0001 C CNN
+F 3 "~" H 3400 6750 50  0001 C CNN
+	1    3400 6750
 	1    0    0    -1
 $EndComp
@@
 L Mechanical:MountingHole MH3
 U 1 1 5BAA4ABC
-P 3250 7300
-F 0 "MH3" H 3350 7346 50  0000 L CNN
-F 1 "MountingHole" H 3350 7255 50  0000 L CNN
-F 2 "MountingHole:MountingHole_3.2mm_M3_ISO14580" H 3250 7300 50  0001 C CNN
-F 3 "~" H 3250 7300 50  0001 C CNN
-	1    3250 7300
+P 2450 7200
+F 0 "MH3" H 2550 7246 50  0000 L CNN
+F 1 "MountingHole" H 2550 7155 50  0000 L CNN
+F 2 "MountingHole:MountingHole_3.2mm_M3_ISO14580" H 2450 7200 50  0001 C CNN
+F 3 "~" H 2450 7200 50  0001 C CNN
+	1    2450 7200
 	1    0    0    -1
 $EndComp
@@
 L Mechanical:MountingHole MH4
 U 1 1 5BAA4BD9
-P 4200 7300
-F 0 "MH4" H 4300 7346 50  0000 L CNN
-F 1 "MountingHole" H 4300 7255 50  0000 L CNN
-F 2 "MountingHole:MountingHole_3.2mm_M3_ISO14580" H 4200 7300 50  0001 C CNN
-F 3 "~" H 4200 7300 50  0001 C CNN
-	1    4200 7300
+P 3400 7200
+F 0 "MH4" H 3500 7246 50  0000 L CNN
+F 1 "MountingHole" H 3500 7155 50  0000 L CNN
+F 2 "MountingHole:MountingHole_3.2mm_M3_ISO14580" H 3400 7200 50  0001 C CNN
+F 3 "~" H 3400 7200 50  0001 C CNN
+	1    3400 7200
 	1    0    0    -1
 $EndComp
 Wire Notes Line
-	3050 6600 3050 7650
+	2250 6500 2250 7550
 Wire Notes Line
-	3050 7650 5000 7650
+	2250 7550 4200 7550
 Wire Notes Line
-	5000 7650 5000 6600
+	4200 7550 4200 6500
 Wire Notes Line
-	5000 6600 3050 6600
-Text Notes 3300 7600 0    50   ~ 10
+	4200 6500 2250 6500
+Text Notes 2500 7500 0    50   ~ 10
 AGUJEROS DE SUJECION DE LA PLACA\n
 Text Notes 1100 7550 0    50   ~ 10

Commit message: Agregado fiduciales, texto en capa de cobre y arreglo de errores
Parts:
- added F1: Fiducial, Fiducial:Fiducial_0.5mm_Dia_1mm_Outer, symbol Mechanical:MountingHole
Other:
- note added: "FIDUCIALES DE \nLA PLACA\n"
Changed lines of the file:
@@
 	2250 6500 2250 7550
 Wire Notes Line
-	2250 7550 4200 7550
-Wire Notes Line
 	4200 7550 4200 6500
-Wire Notes Line
-	4200 6500 2250 6500
 Text Notes 2500 7500 0    50   ~ 10
 AGUJEROS DE SUJECION DE LA PLACA\n
@@
 	1    0    0    -1
 $EndComp
+$Comp
+L Mechanical:MountingHole F1
+U 1 1 5BC35A07
+P 4500 7000
+F 0 "F1" H 4600 7046 50  0000 L CNN
+F 1 "Fiducial" H 4600 6955 50  0000 L CNN
+F 2 "Fiducial:Fiducial_0.5mm_Dia_1mm_Outer" H 4500 7000 50  0001 C CNN
+F 3 "~" H 4500 7000 50  0001 C CNN
+	1    4500 7000
+	1    0    0    -1
+$EndComp
+Wire Notes Line
+	5000 6500 5000 7550
+Wire Notes Line
+	2250 7550 5000 7550
+Wire Notes Line
+	2250 6500 5000 6500
+Text Notes 4350 7500 0    50   ~ 10
+FIDUCIALES DE \nLA PLACA\n
 $EndSCHEMATC

Commit message: Arreglos de revision - Problema persistente: No es posible visualizar huella propia de los reles
Parts:
- J10: value Conn_01x03 -> Tira de Pines Macho
Other:
- note added: "IMPORTANTE: Las entradas son activas en bajo"

Commit message: Error footprint propio solucionado
Parts:
- K1, K2, K3, K4, K5, K6, K7, K8: footprint Relay_THT:Relay_SPDT_SONGLE_SRD_Series_Form_C -> SONGLE_THT:Relay_SPDT_SONGLE_SRD_Series_Form_C
Changed lines of the file:
@@
 F 0 "K1" H 4250 1850 50  0000 L CNN
 F 1 "SONGLE_SRD_Form_C" H 3950 1750 50  0000 L CNN
-F 2 "Relay_THT:Relay_SPDT_SONGLE_SRD_Series_Form_C" H 4700 1250 50  0001 L CNN
-F 3 "http://www.sanyourelay.ca/public/products/pdf/SRD.pdf" H 4250 1300 50  0001 C CNN
+F 2 "SONGLE_THT:Relay_SPDT_SONGLE_SRD_Series_Form_C" H 4700 1250 50  0001 L CNN
+F 3 "http://www.circuitbasics.com/wp-content/uploads/2015/11/SRD-05VDC-SL-C-Datasheet.pdf" H 4250 1300 50  0001 C CNN
 	1    4250 1300
 	1    0    0    -1
@@
 F 0 "K2" H 9000 1850 50  0000 L CNN
 F 1 "SONGLE_SRD_Form_C" H 8700 1750 50  0000 L CNN
-F 2 "Relay_THT:Relay_SPDT_SONGLE_SRD_Series_Form_C" H 9450 1250 50  0001 L CNN
-F 3 "http://www.sanyourelay.ca/public/products/pdf/SRD.pdf" H 9000 1300 50  0001 C CNN
+F 2 "SONGLE_THT:Relay_SPDT_SONGLE_SRD_Series_Form_C" H 9450 1250 50  0001 L CNN
+F 3 "http://www.circuitbasics.com/wp-content/uploads/2015/11/SRD-05VDC-SL-C-Datasheet.pdf" H 9000 1300 50  0001 C CNN
 	1    9000 1300
 	1    0    0    -1
@@
 F 0 "K3" H 2950 3950 50  0000 L CNN
 F 1 "SONGLE_SRD_Form_C" H 2650 3850 50  0000 L CNN
-F 2 "Relay_THT:Relay_SPDT_SONGLE_SRD_Series_Form_C" H 3400 3350 50  0001 L CNN
-F 3 "http://www.sanyourelay.ca/public/products/pdf/SRD.pdf" H 2950 3400 50  0001 C CNN
+F 2 "SONGLE_THT:Relay_SPDT_SONGLE_SRD_Series_Form_C" H 3400 3350 50  0001 L CNN
+F 3 "http://www.circuitbasics.com/wp-content/uploads/2015/11/SRD-05VDC-SL-C-Datasheet.pdf" H 2950 3400 50  0001 C CNN
 	1    2950 3400
 	1    0    0    -1
@@
 F 0 "K4" H 6350 3950 50  0000 L CNN
 F 1 "SONGLE_SRD_Form_C" H 6050 3850 50  0000 L CNN
-F 2 "Relay_THT:Relay_SPDT_SONGLE_SRD_Series_Form_C" H 6800 3350 50  0001 L CNN
-F 3 "http://www.sanyourelay.ca/public/products/pdf/SRD.pdf" H 6350 3400 50  0001 C CNN
+F 2 "SONGLE_THT:Relay_SPDT_SONGLE_SRD_Series_Form_C" H 6800 3350 50  0001 L CNN
+F 3 "http://www.circuitbasics.com/wp-content/uploads/2015/11/SRD-05VDC-SL-C-Datasheet.pdf" H 6350 3400 50  0001 C CNN
 	1    6350 3400
 	1    0    0    -1
@@
 F 0 "K5" H 9800 3950 50  0000 L CNN
 F 1 "SONGLE_SRD_Form_C" H 9500 3850 50  0000 L CNN
-F 2 "Relay_THT:Relay_SPDT_SONGLE_SRD_Series_Form_C" H 10250 3350 50  0001 L CNN
-F 3 "http://www.sanyourelay.ca/public/products/pdf/SRD.pdf" H 9800 3400 50  0001 C CNN
+F 2 "SONGLE_THT:Relay_SPDT_SONGLE_SRD_Series_Form_C" H 10250 3350 50  0001 L CNN
+F 3 "http://www.circuitbasics.com/wp-content/uploads/2015/11/SRD-05VDC-SL-C-Datasheet.pdf" H 9800 3400 50  0001 C CNN
 	1    9800 3400
 	1    0    0    -1
@@
 F 0 "K6" H 2950 5750 50  0000 L CNN
 F 1 "SONGLE_SRD_Form_C" H 2650 5650 50  0000 L CNN
-F 2 "Relay_THT:Relay_SPDT_SONGLE_SRD_Series_Form_C" H 3400 5150 50  0001 L CNN
-F 3 "http://www.sanyourelay.ca/public/products/pdf/SRD.pdf" H 2950 5200 50  0001 C CNN
+F 2 "SONGLE_THT:Relay_SPDT_SONGLE_SRD_Series_Form_C" H 3400 5150 50  0001 L CNN
+F 3 "http://www.circuitbasics.com/wp-content/uploads/2015/11/SRD-05VDC-SL-C-Datasheet.pdf" H 2950 5200 50  0001 C CNN
 	1    2950 5200
 	1    0    0    -1
@@
 F 0 "K8" H 9800 5750 50  0000 L CNN
 F 1 "SONGLE_SRD_Form_C" H 9500 5650 50  0000 L CNN
-F 2 "Relay_THT:Relay_SPDT_SONGLE_SRD_Series_Form_C" H 10250 5150 50  0001 L CNN
-F 3 "http://www.sanyourelay.ca/public/products/pdf/SRD.pdf" H 9800 5200 50  0001 C CNN
+F 2 "SONGLE_THT:Relay_SPDT_SONGLE_SRD_Series_Form_C" H 10250 5150 50  0001 L CNN
+F 3 "http://www.circuitbasics.com/wp-content/uploads/2015/11/SRD-05VDC-SL-C-Datasheet.pdf" H 9800 5200 50  0001 C CNN
 	1    9800 5200
 	1    0    0    -1
@@
 F 0 "K7" H 6350 5750 50  0000 L CNN
 F 1 "SONGLE_SRD_Form_C" H 6050 5650 50  0000 L CNN
-F 2 "Relay_THT:Relay_SPDT_SONGLE_SRD_Series_Form_C" H 6800 5150 50  0001 L CNN
-F 3 "http://www.sanyourelay.ca/public/products/pdf/SRD.pdf" H 6350 5200 50  0001 C CNN
+F 2 "SONGLE_THT:Relay_SPDT_SONGLE_SRD_Series_Form_C" H 6800 5150 50  0001 L CNN
+F 3 "http://www.circuitbasics.com/wp-content/uploads/2015/11/SRD-05VDC-SL-C-Datasheet.pdf" H 6350 5200 50  0001 C CNN
 	1    6350 5200
 	1    0    0    -1

Commit message: Arreglos luego de la revision del profesor
Parts:
- added F1, F3: Fiducial, Fiducial:Fiducial_0.5mm_Dia_1mm_Outer, symbol Mechanical:MountingHole
- D1, D2, D3, D4, D5, D6, D7, D8: Catalogo (none) -> http://www.microelectronicash.com/1n4148smd--det--1N4148SMD
- IN1, IN2, IN3, IN4, IN5, IN6, IN7, IN8: Catalogo (none) -> http://www.microelectronicash.com/l-1206r--det--L-1206R
- J1, J10, J2, J3, J4, J5, J6, J7, J8, J9: Catalogo (none) -> http://www.microelectronicash.com/tp1x20-2-00--det--TP1X20-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
- K1, K2, K3, K4, K5, K7, K8: Catalogo (none) -> https://candy-ho.com/producto/modulo-rele-5v-simple-inverso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
- Q1, Q2, Q3, Q4, Q5, Q6, Q7, Q8: Catalogo (none) -> https://www.digikey.com/product-detail/en/micro-commercial-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
- R1, R11, R13, R15, R3, R5, R7, R9: Catalogo (none) -> http://www.microelectronicash.com/r1206-1k--det--R1206-1K
- U1, U2, U3, U4, U5, U6, U7, U8: Catalogo (none) -> https://www.digikey.com/product-detail/es/sharp-socle-techn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
- renumbered F1 to F2
Connections:
- net labels added: VCC
- net labels removed: JD-VCC
- wire segments 293 -> 288
